File: PCB/compass.kicad_pcb (KiCad board)
At the start: 2 copper layers, 82.5 x 85 mm, 89 parts, among them Q1 BSS138, U1 XIAO-RP2040-DIP

Commit message: bruh
Parts:
- added JP1: SolderJumper_2_Bridged, Jumper:SolderJumper-2_P1.3mm_Bridged_RoundedPad1.0x1.5mm, B.Cu at (85.5, 83.3)
- added JP2: SolderJumper_3_Bridged12, Jumper:SolderJumper-3_P1.3mm_Bridged12_RoundedPad1.0x1.5mm, B.Cu at (83.0, 82.5)
- added JP3: SolderJumper_3_Bridged12, Jumper:SolderJumper-3_P1.3mm_Bridged12_RoundedPad1.0x1.5mm, B.Cu at (80.5, 82.5)
- added JP4: SolderJumper_3_Bridged123, Jumper:SolderJumper-3_P1.3mm_Bridged123_RoundedPad1.0x1.5mm_NumberLabels, B.Cu at (85.5, 79.0)
- added R3: 10K, Resistor_SMD:R_0603_1608Metric_Pad0.98x0.95mm_HandSolder, B.Cu at (79.7, 77.5)
- added R4: 10K, Resistor_SMD:R_0603_1608Metric_Pad0.98x0.95mm_HandSolder, B.Cu at (79.7, 79.0)
- added U2: MLX90395xLW, Package_DFN_QFN:QFN-16-1EP_3x3mm_P0.5mm_EP1.675x1.675mm, B.Cu at (76.0, 72.0)
Connections:
- U1 pad 1: unconnected-(U1-GPIO26/ADC0/A0-Pad1) -> CS
- U1 pad 10: unconnected-(U1-GPIO4/MISO-Pad10) -> MISO
- U1 pad 11: unconnected-(U1-GPIO3/MOSI-Pad11) -> SDA
- U1 pad 2: unconnected-(U1-GPIO27/ADC1/A1-Pad2) -> TRIG
- U1 pad 3: unconnected-(U1-GPIO28/ADC2/A2-Pad3) -> INT
- U1 pad 5: unconnected-(U1-GPIO6/SDA-Pad5) -> SDA
- U1 pad 6: unconnected-(U1-GPIO7/SCL-Pad6) -> SCL
Routing:
- net LV: track 1.88 -> 70.2 mm, vias 0 -> 1
- net CS: track 0.00 -> 50.8 mm, vias 0 -> 2
- net SDA: track 0.00 -> 37.6 mm
- net TRIG: track 0.00 -> 35.0 mm
- net VBUS: track 470.6 -> 502.6 mm, vias 0 -> 2
- net SCL: track 0.00 -> 27.0 mm, vias 0 -> 1
- net INT: track 0.00 -> 24.7 mm, vias 0 -> 1
- net A0: track 0.00 -> 15.7 mm, vias 0 -> 2
- net A1: track 0.00 -> 12.9 mm, vias 0 -> 2
- net LED_LV: track 4.49 -> 10.0 mm
- net Net-(JP4-A): track 0.00 -> 5.38 mm
- net Net-(JP4-B): track 0.00 -> 4.92 mm
- net unconnected-(U1-GPIO7/SCL-Pad6): track 0.84 -> 0.00 mm
- net (no net): track 0.00 -> 0.84 mm
- net GND: track 5.69 -> 4.85 mm, vias 70 -> 68
