File: PCB/compass.kicad_sch (KiCad schematic)
At the start: 84 parts, among them Q1 BSS138, U1 XIAO-RP2040-DIP

Commit message: bruh
Parts:
- added JP1: SolderJumper_2_Bridged, Jumper:SolderJumper-2_P1.3mm_Bridged_RoundedPad1.0x1.5mm, symbol Jumper:SolderJumper_2_Bridged
- added JP2, JP3: SolderJumper_3_Bridged12, Jumper:SolderJumper-3_P1.3mm_Bridged12_RoundedPad1.0x1.5mm, symbol Jumper:SolderJumper_3_Bridged12
- added JP4: SolderJumper_3_Bridged123, Jumper:SolderJumper-3_P1.3mm_Bridged123_RoundedPad1.0x1.5mm_NumberLabels, symbol Jumper:SolderJumper_3_Bridged123
- added R3, R4: 10K, Resistor_SMD:R_0603_1608Metric_Pad0.98x0.95mm_HandSolder, symbol Device:R_US
- added U2: MLX90395xLW, Package_DFN_QFN:QFN-16-1EP_3x3mm_P0.5mm_EP1.675x1.675mm, symbol Sensor_Magnetic:MLX90395xLW
Connections:
- net GND: now also JP2.3 (B), JP3.3 (B), U2.10 (V_{SS}), U2.13 (V_{SS}), U2.14 (V_{SS}), U2.16 (V_{SS}), U2.17 (V_{SS}), U2.4 (V_{SS}), U2.8 (V_{SS}), U2.9 (V_{SS})
- net LV: now also JP1.2 (B), JP2.1 (A), JP3.1 (A), JP4.2 (C), U2.15 (V_{DD})
- net CS: now reaches U1.1 (GPIO26/ADC0/A0)
- net CS: now also JP1.1 (A), U2.2 (~{CS})
- net MISO: now reaches U1.10 (GPIO4/MISO)
- net MISO: now also U2.6 (MISO)
- net SDA: now reaches U1.11 (GPIO3/MOSI)
- net SDA: now also U1.5 (GPIO6/SDA), R4.1, U2.5 (MOSI)
- net TRIG: now reaches U1.2 (GPIO27/ADC1/A1)
- net TRIG: now also U2.7 (INT/TRG)
- net INT: now reaches U1.3 (GPIO28/ADC2/A2)
- net INT: now also U2.1 (INT)
- net SCL: now reaches U1.6 (GPIO7/SCL)
- net SCL: now also R3.1, U2.3 (SCLK)
- new net: JP4.3 (B), R3.2
- new net: JP4.1 (A), R4.2
- new net A0: JP2.2 (C), U2.11 (A1)
- new net A1: JP3.2 (C), U2.12 (A0)
